File: qx3/qx3.kicad_pcb (KiCad board)
At the start: 2 copper layers, 121 parts, among them J1 TYPE-C-31-M12_13, Q1 DTC123J, SW1 SHIFT▲, SW10 ., SW11 _, SW12 !, SW13 ?, SW14 &, SW15 F1, SW16 F2, SW17 U, SW18 V, SW19 W, SW2 CHAR, SW20 X, SW21 Y, SW22 Z, SW23 +, SW24 -, SW25 *, SW26 /, SW27 K, SW28 L, SW29 M, SW3 ENTER, SW30 N, SW31 O, SW32 P, SW33 Q, SW34 R, SW35 S, SW36 T, SW37 A, SW38 B, SW39 C, SW4 JOB COMMAND, SW40 D, SW41 E, SW42 F, SW43 G, SW44 H, SW45 I, SW46 J, SW5 ◀, SW6 ▶, SW7 INS, SW8 (, SW9 ), U1 STM32F072-LQFP48, U2 USBLC6-2SC6, U3 MCP1700-3302E_SOT23

Commit message: Update QX3
Parts:
- J1: footprint Type-C:HRO-TYPE-C-31-M-12 -> Type-C:HRO-TYPE-C-31-M-12-HandSoldering
- SW3: footprint MX_Only:MXOnly-1U-Hotswap -> MXOnly-4U-Hotswap:MXOnly-4U-Hotswap
- moved J1 316.7 mm to (221.9, 59.3), turned to 180 degrees
- turned SW45 to 180 degrees
- turned SW46 to 180 degrees
