File: qx3/qx3.sch (KiCad schematic (older format))
At the start: 121 parts, among them J1 TYPE-C-31-M12_13, Q1 DTC123J, SW1 SHIFT▲, SW10 ., SW11 _, SW12 !, SW13 ?, SW14 &, SW15 F1, SW16 F2, SW17 U, SW18 V, SW19 W, SW2 CHAR, SW20 X, SW21 Y, SW22 Z, SW23 +, SW24 -, SW25 *, SW26 /, SW27 K, SW28 L, SW29 M, SW3 ENTER, SW30 N, SW31 O, SW32 P, SW33 Q, SW34 R, SW35 S, SW36 T, SW37 A, SW38 B, SW39 C, SW4 JOB COMMAND, SW40 D, SW41 E, SW42 F, SW43 G, SW44 H, SW45 I, SW46 J, SW5 ◀, SW6 ▶, SW7 INS, SW8 (, SW9 ), U1 STM32F072-LQFP48, U2 USBLC6-2SC6, U3 MCP1700-3302E_SOT23

Commit message: Update QX3
Parts:
- J1: footprint Type-C:HRO-TYPE-C-31-M-12 -> Type-C:HRO-TYPE-C-31-M-12-HandSoldering
- SW3: footprint MX_Only:MXOnly-1U-Hotswap -> MXOnly-4U-Hotswap:MXOnly-4U-Hotswap
Changed lines of the file:
@@
 F 0 "J1" H 6967 3872 50  0000 C CNN
 F 1 "TYPE-C-31-M12_13" H 6967 3781 50  0000 C CNN
-F 2 "Type-C:HRO-TYPE-C-31-M-12" V 6360 2505 50  0001 C CNN
+F 2 "Type-C:HRO-TYPE-C-31-M-12-HandSoldering" V 6360 2505 50  0001 C CNN
 F 3 "" H 7060 2505 50  0001 C CNN
 	1    6860 2455
@@
 F 0 "SW3" H 7025 12135 50  0000 L CNN
 F 1 "ENTER" H 6980 12070 39  0000 L CNN
-F 2 "MX_Only:MXOnly-1U-Hotswap" H 7100 12080 50  0001 C CNN
+F 2 "MXOnly-4U-Hotswap:MXOnly-4U-Hotswap" H 7100 12080 50  0001 C CNN
 F 3 "" H 7100 12080 50  0001 C CNN
 	1    7100 12080
